Commit message: update

File: ar_description/urdf/ar.urdf.xacro (robot description, xacro)
@@ -1,4 +1,4 @@
 <?xml version="1.0"?>
-<robot xmlns:xacro="http://wiki.ros.org/xacro" name="ar4">
+<robot xmlns:xacro="http://wiki.ros.org/xacro" name="$(arg name)">
   <xacro:include filename="$(find ar_description)/urdf/ar_macro.xacro"/>
   <link name="world" />

File: ar_description/urdf/ar_macro.xacro (robot description, xacro)
@@ -4,5 +4,4 @@
     <joint name="base_joint" type="fixed">
       <xacro:insert_block name="origin" />
-     <origin rpy="${pi/2} 0 0" xyz="0 0 0"/>
      <parent link="${parent}"/>
       <child link="base_link" />
@@ -20,5 +19,5 @@
         </geometry>
         <material name="">
-          <color rgba="1 1 0 0.1"/>
+          <color rgba="1 1 0 1"/>
         </material>
       </visual>
@@ -42,5 +41,5 @@
         </geometry>
         <material name="">
-          <color rgba="1 1 0 0.1"/>
+          <color rgba="1 1 0 1"/>
         </material>
       </visual>
@@ -71,5 +70,5 @@
         </geometry>
         <material name="">
-          <color rgba="1 1 0 0.1"/>
+          <color rgba="1 1 0 1"/>
         </material>
       </visual>
@@ -100,5 +99,5 @@
         </geometry>
         <material name="">
-          <color rgba="1 1 0 0.1"/>
+          <color rgba="1 1 0 1"/>
         </material>
       </visual>
@@ -129,5 +128,5 @@
         </geometry>
         <material name="">
-          <color rgba="1 1 0 0.1"/>
+          <color rgba="1 1 0 1"/>
         </material>
       </visual>
@@ -158,5 +157,5 @@
         </geometry>
         <material name="">
-          <color rgba="1 1 0 0.1"/>
+          <color rgba="1 1 0 1"/>
         </material>
       </visual>
@@ -187,5 +186,5 @@
         </geometry>
         <material name="">
-          <color rgba="1 1 0 0.1"/>
+          <color rgba="1 1 0 1"/>
         </material>
       </visual>
