Commit message: imported solid works and keninmatics are modified to work

File: ar_description/urdf/ar_macro.xacro (robot description, xacro)
@@ -4,5 +4,6 @@
     <joint name="base_joint" type="fixed">
       <xacro:insert_block name="origin" />
-      <parent link="${parent}"/>
+     <origin rpy="${pi/2} 0 0" xyz="0 0 0"/>
+     <parent link="${parent}"/>
       <child link="base_link" />
     </joint>
@@ -14,10 +15,10 @@
       </inertial>
       <visual>
-        <origin rpy="0 0 0" xyz="0 0 0"/>
+        <origin rpy="${pi/2} 0 0" xyz="0 0 0"/>
         <geometry>
           <mesh filename="file://$(find ar_description)/meshes/ar4/base_link.STL"/>
         </geometry>
         <material name="">
-          <color rgba="1 1 0 1"/>
+          <color rgba="1 1 0 0.1"/>
         </material>
       </visual>
@@ -41,5 +42,5 @@
         </geometry>
         <material name="">
-          <color rgba="1 1 0 1"/>
+          <color rgba="1 1 0 0.1"/>
         </material>
       </visual>
@@ -52,27 +53,27 @@
     </link>
     <joint name="joint_1" type="revolute">
-      <origin rpy="${pi} 0 0" xyz="0 0 0.003445"/>
+      <origin rpy="${pi/2} 0 0" xyz="0 0 0"/>
       <parent link="base_link"/>
       <child link="link_1"/>
-      <axis xyz="0 0 1"/>
+      <axis xyz="0 1 0"/>
       <limit lower="${-170.0 / 180.0 * pi}" upper="${170.0 / 180.0 * pi}" effort="0" velocity="0.5"/>
     </joint>
     <link name="link_2">
       <inertial>
-        <origin rpy="0 0 0" xyz="0.064818 -0.11189 -0.038671"/>
+        <origin rpy="0 0 0" xyz="0.06384 -0.1736 -0.038671"/>
         <mass value="0.57738"/>
         <inertia ixx="0.0047312" ixy="0.0022624" ixz="0.00032144" iyy="0.0020836" iyz="-0.00056569" izz="0.0056129"/>
       </inertial>
       <visual>
-        <origin rpy="0 0 0" xyz="0 0 0"/>
+        <origin rpy="0 0 ${pi}" xyz="0 0 0"/>
         <geometry>
           <mesh filename="file://$(find ar_description)/meshes/ar4/link_2.STL"/>
         </geometry>
         <material name="">
-          <color rgba="1 1 0 1"/>
-        </material>
-      </visual>
-      <collision>
-        <origin rpy="0 0 0" xyz="0 0 0"/>
+          <color rgba="1 1 0 0.1"/>
+        </material>
+      </visual>
+      <collision>
+        <origin rpy="0 0 ${pi}" xyz="0 0 0"/>
         <geometry>
           <mesh filename="file://$(find ar_description)/meshes/ar4/link_2.STL"/>
@@ -81,8 +82,8 @@
     </link>
     <joint name="joint_2" type="revolute">
-      <origin rpy="1.5708 0.5236 -1.5708" xyz="0 0.064146 -0.16608"/>
+      <origin rpy="0 0 ${pi}" xyz="0.06384 0.1736 0"/>
       <parent link="link_1"/>
       <child link="link_2"/>
-      <axis xyz="0 0 -1"/>
+      <axis xyz="0 0 1"/>
       <limit lower="${-42.0 / 180.0 * pi}" upper="${90.0 / 180.0 * pi}" effort="0.5" velocity="0"/>
     </joint>
@@ -99,5 +100,5 @@
         </geometry>
         <material name="">
-          <color rgba="1 1 0 1"/>
+          <color rgba="1 1 0 0.1"/>
         </material>
       </visual>
@@ -110,5 +111,5 @@
     </link>
     <joint name="joint_3" type="revolute">
-      <origin rpy="0 0 -2.61799" xyz="0.1525 -0.26414 0"/>
+      <origin rpy="0 0 ${pi}" xyz="0 -0.34997 0.0046"/>
       <parent link="link_2"/>
       <child link="link_3"/>
@@ -128,5 +129,5 @@
         </geometry>
         <material name="">
-          <color rgba="1 1 0 1"/>
+          <color rgba="1 1 0 0.1"/>
         </material>
       </visual>
@@ -139,8 +140,8 @@
     </link>
     <joint name="joint_4" type="revolute">
-      <origin rpy="1.5708 -1.2554 -1.5708" xyz="0 0 0.00675"/>
+      <origin rpy="0 0 0" xyz="0 0 0"/>
       <parent link="link_3"/>
       <child link="link_4"/>
-      <axis xyz="0 0 -1"/>
+      <axis xyz="1 0 0"/>
       <limit lower="${-165.0 / 180.0 * pi}" upper="${165.0 / 180.0 * pi}" effort="0" velocity="0.5"/>
     </joint>
@@ -157,5 +158,5 @@
         </geometry>
         <material name="">
-          <color rgba="1 1 0 1"/>
+          <color rgba="1 1 0 0.1"/>
         </material>
       </visual>
@@ -168,8 +169,8 @@
     </link>
     <joint name="joint_5" type="revolute">
-      <origin rpy="${pi} 0 -2.8262" xyz="0 0 -0.22225"/>
+      <origin rpy="0 0 0" xyz="0.27435 0 0"/>
       <parent link="link_4"/>
       <child link="link_5"/>
-      <axis xyz="1 0 0"/>
+      <axis xyz="0 0 -1"/>
       <limit lower="${-105.0 / 180.0 * pi}" upper="${105.0 / 180.0 * pi}" effort="0" velocity="0.5"/>
     </joint>
@@ -186,5 +187,5 @@
         </geometry>
         <material name="">
-          <color rgba="1 1 0 1"/>
+          <color rgba="1 1 0 0.1"/>
         </material>
       </visual>
@@ -197,8 +198,8 @@
     </link>
     <joint name="joint_6" type="revolute">
-      <origin rpy="0 0 3.1416" xyz="-0.000294 0 0.02117"/>
+      <origin rpy="0 0 0" xyz="0.0384 0 0"/>
       <parent link="link_5"/>
       <child link="link_6"/>
-      <axis xyz="0 0 1"/>
+      <axis xyz="1 0 0"/>
       <limit lower="${-155.0 / 180.0 * pi}" upper="${155.0 / 180.0 * pi}" effort="0" velocity="0.5"/>
     </joint>

Commit message: timeout change and limits

File: ar_description/urdf/ar_macro.xacro (robot description, xacro)
@@ -55,6 +55,6 @@
       <parent link="base_link"/>
       <child link="link_1"/>
-      <axis xyz="0 1 0"/>
-      <limit lower="${-170.0 / 180.0 * pi}" upper="${170.0 / 180.0 * pi}" effort="0" velocity="0.5"/>
+      <axis xyz="0 -1 0"/>
+      <limit lower="${-184.0 / 180.0 * pi}" upper="${150.0 / 180.0 * pi}" effort="0" velocity="0.5"/>
     </joint>
     <link name="link_2">
@@ -84,6 +84,6 @@
       <parent link="link_1"/>
       <child link="link_2"/>
-      <axis xyz="0 0 1"/>
-      <limit lower="${-42.0 / 180.0 * pi}" upper="${90.0 / 180.0 * pi}" effort="0.5" velocity="0"/>
+      <axis xyz="0 0 -1"/>
+      <limit lower="${-47.0 / 180.0 * pi}" upper="${120.0 / 180.0 * pi}" effort="0.5" velocity="0"/>
     </joint>
     <link name="link_3">
@@ -114,5 +114,5 @@
       <child link="link_3"/>
       <axis xyz="0 0 -1"/>
-      <limit lower="${-89.0 / 180.0 * pi}" upper="${52.0 / 180.0 * pi}" effort="0" velocity="0.5"/>
+      <limit lower="${-110.0 / 180.0 * pi}" upper="${62.0 / 180.0 * pi}" effort="0" velocity="0.5"/>
     </joint>
     <link name="link_4">
@@ -143,5 +143,5 @@
       <child link="link_4"/>
       <axis xyz="1 0 0"/>
-      <limit lower="${-165.0 / 180.0 * pi}" upper="${165.0 / 180.0 * pi}" effort="0" velocity="0.5"/>
+      <limit lower="${-177.0 / 180.0 * pi}" upper="${161.0 / 180.0 * pi}" effort="0" velocity="0.5"/>
     </joint>
     <link name="link_5">
@@ -172,5 +172,5 @@
       <child link="link_5"/>
       <axis xyz="0 0 -1"/>
-      <limit lower="${-105.0 / 180.0 * pi}" upper="${105.0 / 180.0 * pi}" effort="0" velocity="0.5"/>
+      <limit lower="${-103.0 / 180.0 * pi}" upper="${103.0 / 180.0 * pi}" effort="0" velocity="0.5"/>
     </joint>
     <link name="link_6">
@@ -201,5 +201,5 @@
       <child link="link_6"/>
       <axis xyz="1 0 0"/>
-      <limit lower="${-155.0 / 180.0 * pi}" upper="${155.0 / 180.0 * pi}" effort="0" velocity="0.5"/>
+      <limit lower="${-167.0 / 180.0 * pi}" upper="${170.0 / 180.0 * pi}" effort="0" velocity="0.5"/>
     </joint>
   </xacro:macro>

Commit message: change 184 to 150

File: ar_description/urdf/ar_macro.xacro (robot description, xacro)
@@ -56,5 +56,5 @@
       <child link="link_1"/>
       <axis xyz="0 -1 0"/>
-      <limit lower="${-184.0 / 180.0 * pi}" upper="${150.0 / 180.0 * pi}" effort="0" velocity="0.5"/>
+      <limit lower="${-150.0 / 180.0 * pi}" upper="${184.0 / 180.0 * pi}" effort="0" velocity="0.5"/>
     </joint>
     <link name="link_2">
